Commit message: removed front L4 tof and rear OPT sensors from sensor node and urdf

File: urdfs/rr26.urdf (robot description, URDF)
Before this commit: robot roborama25, 15 links, 14 joints
Links:
- removed link tofL4_link
- removed link tofRC_link
- removed link tofRL_link
- removed link tofRR_link
Joints:
- removed joint tofL4_joint
- removed joint tofRC_joint
- removed joint tofRL_joint
- removed joint tofRR_joint

Commit message: Scaled battery voltage correctly Use opnemv blob height to determine distance. Use blob horozntal location and distance to detrmine the map XY coordinates of the detected can.

File: urdfs/rr26.urdf (robot description, URDF)
Before this commit: robot rr26, 11 links, 10 joints
Links:
- added link cam_link; visual box size=0.025 0.025 0.015
Joints:
- added joint cam_joint: type fixed, parent base_link, child cam_link, origin xyz=0.070 0 0.050 rpy=0 0 0
- joint lidar_joint: origin xyz=0 0 0.115 rpy=0 0 3.1416 -> xyz=0 0 0.075 rpy=0 0 3.1416

Commit message: lidar: physically change the lidar direction -180 deg which "fixes" the discontinuity (begin-end- scannin g) of the scan data in front of the robot and moves the distortion to behind the robot. Adjusted urdf and the lidar can node with the new orientation

File: urdfs/rr26.urdf (robot description, URDF)
Before this commit: robot rr26, 11 links, 10 joints
Joints:
- joint lidar_joint: origin xyz=0 0 0.075 rpy=0 0 3.1416 -> xyz=0 0 0.075 rpy=0 0 0
